Commit message: Modernize repo: hygiene, cross-platform paths, packaging, docs
- Add proper .gitignore; remove committed orphan .pyc artifact
- Add requirements.txt and pyproject.toml (no dependency manifest existed)
- YertleUI.py: resolve config/URDF paths via pathlib (cross-platform, run from any cwd); replace bare assert with clear FileNotFoundError
- yertle.URDF: fix 19 mesh paths to be relative to the URDF file and use forward slashes
- Rename 'yertle lib.{h,cpp}' to yertle_lib.{h,cpp} and update includes; fix EPS32 typo
- README: add repository structure and getting-started sections; fix WiFi password and file-location errors

File: Simulation/yertle.URDF (robot description, URDF)
Before this commit: robot Dog, 14 links, 13 joints
Links:
- link base_link: geometry visual mesh filename=URDF/frame.obj
- link frame: geometry collision mesh filename=URDF/shell.obj; visual mesh filename=URDF/shell.obj
- link lb_shin: geometry collision mesh filename=URDF/tibia.obj; visual mesh filename=URDF/tibia.obj
- link lb_shoulder: geometry visual mesh filename=URDF/lb shoulder.obj
- link lb_thigh: geometry visual mesh filename=URDF/femur.obj
- link lf_shin: geometry collision mesh filename=URDF/tibia.obj; visual mesh filename=URDF/tibia.obj
- link lf_shoulder: geometry visual mesh filename=URDF/lf shoulder.obj
- link lf_thigh: geometry visual mesh filename=URDF/femur.obj
- link rb_shin: geometry collision mesh filename=URDF/tibia.obj; visual mesh filename=URDF/tibia.obj
- link rb_shoulder: geometry visual mesh filename=URDF/rb shoulder.obj
- link rb_thigh: geometry visual mesh filename=URDF/femur.obj
- link rf_shin: geometry collision mesh filename=URDF/tibia.obj; visual mesh filename=URDF/tibia.obj
- link rf_shoulder: geometry visual mesh filename=URDF/rf shoulder.obj
- link rf_thigh: geometry visual mesh filename=URDF/femur.obj

Commit message: Fix robot model: valid inertia tensors, no-space mesh filenames
- Replace the URDF's invalid inertia tensors (zeros on base, off-diagonal
  equal to diagonal on legs) with valid mass-scaled diagonal tensors; PhysX
  rejects the originals for articulations
- Rename the four 'x shoulder' mesh files to 'x_shoulder' and fix mtllib refs;
  spaces are illegal in USD prim paths
- gitignore generated Simulation/usd/ and isaac_lab/runs/

File: Simulation/yertle.URDF (robot description, URDF)
Before this commit: robot Dog, 14 links, 13 joints
Links:
- link lb_shoulder: geometry visual mesh filename=URDF/lb_shoulder.obj
- link lf_shoulder: geometry visual mesh filename=URDF/lf_shoulder.obj
- link rb_shoulder: geometry visual mesh filename=URDF/rb_shoulder.obj
- link rf_shoulder: geometry visual mesh filename=URDF/rf_shoulder.obj

Commit message: Add firmware joint limits and actuator caps to the simulation model
- URDF: 12 leg joints continuous -> revolute with firmware-derived limits
  (shoulder +/-45deg, thigh -90..20deg, shin 13..90deg), effort 3 N.m,
  velocity 10 rad/s; PhysX now enforces them as hard constraints
- Keep the implicit PhysX drive with effort/velocity caps: an explicit
  DC-motor model was tried and is underdamped at hobby-servo gains (the
  robot oscillates against its limits and cannot hold stance); reasoning
  documented in yertle_cfg.py
- Flat-task reward: gentle smoothness shaping (action rate, body wobble,
  joint-limit proximity) tuned so per-step reward of useful behavior stays
  positive; heavier penalties made falling immediately the optimal policy

File: Simulation/yertle.URDF (robot description, URDF)
Before this commit: robot Dog, 14 links, 13 joints
Joints:
- joint lb_shin: limit (none) -> lower=0.2269 upper=1.5708 effort=3.0 velocity=10.0; type continuous -> revolute
- joint lb_shoulder: limit (none) -> lower=-0.7854 upper=0.7854 effort=3.0 velocity=10.0; type continuous -> revolute
- joint lb_thigh: limit (none) -> lower=-1.5708 upper=0.3491 effort=3.0 velocity=10.0; type continuous -> revolute
- joint lf_shin: limit (none) -> lower=0.2269 upper=1.5708 effort=3.0 velocity=10.0; type continuous -> revolute
- joint lf_shoulder: limit (none) -> lower=-0.7854 upper=0.7854 effort=3.0 velocity=10.0; type continuous -> revolute
- joint lf_thigh: limit (none) -> lower=-1.5708 upper=0.3491 effort=3.0 velocity=10.0; type continuous -> revolute
- joint rb_shin: limit (none) -> lower=0.2269 upper=1.5708 effort=3.0 velocity=10.0; type continuous -> revolute
- joint rb_shoulder: limit (none) -> lower=-0.7854 upper=0.7854 effort=3.0 velocity=10.0; type continuous -> revolute
- joint rb_thigh: limit (none) -> lower=-1.5708 upper=0.3491 effort=3.0 velocity=10.0; type continuous -> revolute
- joint rf_shin: limit (none) -> lower=0.2269 upper=1.5708 effort=3.0 velocity=10.0; type continuous -> revolute
- joint rf_shoulder: limit (none) -> lower=-0.7854 upper=0.7854 effort=3.0 velocity=10.0; type continuous -> revolute
- joint rf_thigh: limit (none) -> lower=-1.5708 upper=0.3491 effort=3.0 velocity=10.0; type continuous -> revolute
