Commit message: Restructure: consistent lowercase layout, snake_case filenames, code polish
Naming was split between the 2022 layout (Design/, Simulation/, Software/,
CamelCase and spaced filenames) and the newer lowercase packages. Unify:

- Design/ -> design/, Simulation/ -> simulation/, Software/ -> software/
- Simulation/yertle.URDF -> simulation/yertle.urdf
- Simulation/URDF/ (meshes) -> simulation/meshes/ (paths inside the URDF
  updated to match)
- Software/YertleUI/YertleUI.py -> software/yertle_ui/yertle_ui.py
- design STL/CAD files: spaces -> underscores (also fixes a double-space
  filename); all bill-of-materials links updated
- every path reference updated (env URDF path, Isaac USD path, bridge, GUI,
  .gitignore, all READMEs); design README also fixes the Right Servo Mount
  row linking to the Left STL, the 150x150cm build-plate typo (mm), and a
  couple of BOM typos

Code polish for readability:
- yertle_ui.py: module docstring, misspelled identifiers fixed
  (YerltleSimulation, balaceMode, curretPosition), blank-line runs collapsed
- firmware: misspelled unused extern instances fixed in yertle_lib.h
  (defalutPoseAngle/defalutPoseCartesian); comment spelling cleaned up in
  yertle_lib.cpp and firmware.ino (no functional changes)

Validated: full python compile, PyBullet smoke test end to end on the
renamed model, and a link check across every README.

File: simulation/yertle.urdf (robot description, URDF)
Before this commit: robot Dog, 14 links, 13 joints
Links:
- link base_link: geometry visual mesh filename=meshes/frame.obj
- link frame: geometry collision mesh filename=meshes/shell.obj; visual mesh filename=meshes/shell.obj
- link lb_shin: geometry collision mesh filename=meshes/tibia.obj; visual mesh filename=meshes/tibia.obj
- link lb_shoulder: geometry visual mesh filename=meshes/lb_shoulder.obj
- link lb_thigh: geometry visual mesh filename=meshes/femur.obj
- link lf_shin: geometry collision mesh filename=meshes/tibia.obj; visual mesh filename=meshes/tibia.obj
- link lf_shoulder: geometry visual mesh filename=meshes/lf_shoulder.obj
- link lf_thigh: geometry visual mesh filename=meshes/femur.obj
- link rb_shin: geometry collision mesh filename=meshes/tibia.obj; visual mesh filename=meshes/tibia.obj
- link rb_shoulder: geometry visual mesh filename=meshes/rb_shoulder.obj
- link rb_thigh: geometry visual mesh filename=meshes/femur.obj
- link rf_shin: geometry collision mesh filename=meshes/tibia.obj; visual mesh filename=meshes/tibia.obj
- link rf_shoulder: geometry visual mesh filename=meshes/rf_shoulder.obj
- link rf_thigh: geometry visual mesh filename=meshes/femur.obj
